File: Solar charger/Solar Charger.kicad_pcb (KiCad board)
At the start: 2 copper layers, 112 x 50 mm, 53 parts, among them J1 Screw_Terminal_01x03, J2 Screw_Terminal_01x02, J3 Screw_Terminal_01x02, P1 USB_C_Plug_USB2.0, U1 CN3795, U2 BW6101_, U3 BW6101_, U4 BW6101_, U5 BW6101_, U6 IP6510

Commit message: compelet
Parts:
- moved R12 65.9 mm to (114.1, 103.8)
- moved U5 59.7 mm to (117.3, 103.9), turned to 180 degrees
- moved C16 53.6 mm to (120.4, 103.9)
- moved C14 46.4 mm to (160.4, 103.9), turned to -90 degrees
- moved C13 26.4 mm to (180.4, 103.9)
- moved U2 20.3 mm to (177.3, 103.9), turned to 180 degrees
- moved U3 20.3 mm to (157.3, 103.9), turned to 180 degrees
- moved U4 20.3 mm to (137.3, 103.9), turned to 180 degrees
- moved R10 14.1 mm to (154.1, 103.8)
- moved R11 14.1 mm to (134.1, 103.8)
- moved R9 14.1 mm to (174.1, 103.8)
- moved C15 6.41 mm to (140.4, 103.9), turned to -90 degrees
- moved C4 3.57 mm to (84.8, 78.3), turned to 0 degrees
- moved C5 2.00 mm to (84.9, 80.4), turned to 180 degrees
- moved R6 0.76 mm to (84.8, 82.4), turned to 0 degrees
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Routing:
- net /IP6510 USB/Power Output: track 0.00 -> 37.3 mm, vias 0 -> 2
- net Net-(C10-Pad2): track 0.00 -> 30.9 mm
- net /CN3795 MPPT/MPPT: track 0.00 -> 29.4 mm, vias 0 -> 2
- net Net-(C11-Pad2): track 0.00 -> 27.1 mm
- net Net-(C10-Pad1): track 0.00 -> 20.0 mm
- net /IP6510 USB/Power Input: track 0.00 -> 19.3 mm, vias 0 -> 10
- net GND: track 0.00 -> 17.9 mm, vias 0 -> 18
- net Net-(D2-Pad1): track 0.00 -> 17.8 mm
- net Net-(D1-Pad1): track 0.00 -> 15.6 mm, vias 0 -> 2
- net Net-(C20-Pad1): track 0.00 -> 13.7 mm
- net Net-(AP1-Pad4): track 0.00 -> 12.3 mm, vias 0 -> 2
- net /CN3795 MPPT/CSP: track 0.00 -> 10.7 mm
- net /CN3795 MPPT/FB: track 0.00 -> 10.7 mm, vias 0 -> 2
- net Net-(J1-Pad1): track 0.00 -> 9.37 mm
- net Net-(AP1-Pad5): track 0.00 -> 7.54 mm
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- added copper zone on F.Cu, net /CN3795 MPPT/BAT
- added copper zone on B.Cu, net /IP6510 USB/Power Input
- added copper zone on F.Cu, net /IP6510 USB/Power Input
- added copper zone on F.Cu, net /IP6510 USB/Power Output
- added copper zone on B.Cu, net GND
- added copper zone on B.Cu, net Net-(C10-Pad1)
- added copper zone on F.Cu, net Net-(C10-Pad1)
- added copper zone on B.Cu, net Net-(C10-Pad2)
- added copper zone on F.Cu, net Net-(C10-Pad2)
- added copper zone on B.Cu, net Net-(C11-Pad2)
- added copper zone on F.Cu, net Net-(C11-Pad2)
- added copper zone on F.Cu, net Net-(J3-Pad2)
- added copper zone on F.Cu, net VCC
Other:
- board size 112 x 50 mm -> 112.3 x 50.3 mm

Commit message: update
Other:
- board text added: "By Andy 2022/08/08"
- board text added: "GND"
- board text added: "MPPT IN"
- board text added: "MPPT OUT"
- board text added: "Solar IN"
- board text added: "Solar OUT"
- board text added: "USB IN"
- board text added: "USB OUT"
- board text added: "VIN"
Changed lines of the file:
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@@
     (property "Sheetname" "IP6510 USB")
     (attr through_hole)
-    (fp_text reference "C21" (at 1.25 -4.4) (layer "F.SilkS")
+    (fp_text reference "C21" (at 4.9 -3.25) (layer "F.SilkS")
       (effects (font (size 1 1) (thickness 0.15)))
     )
@@
   )
   (gr_rect (start 74.05 56.2) (end 186.3 106.55) (layer "Edge.Cuts") (width 0.1) (fill none))
+  (gr_text "MPPT\nIN" (at 82.1 76.1 270) (layer "B.SilkS")
+    (effects (font (size 1.4 1.4) (thickness 0.15)) (justify mirror))
+  )
+  (gr_text "USB\nIN" (at 81.9 88.1 270) (layer "B.SilkS")
+    (effects (font (size 1.4 1.4) (thickness 0.15)) (justify mirror))
+  )
+  (gr_text "MPPT\nOUT" (at 82.05 82.05 270) (layer "B.SilkS")
+    (effects (font (size 1.4 1.4) (thickness 0.15)) (justify mirror))
+  )
+  (gr_text "GND" (at 80.9 64.55 270) (layer "B.SilkS")
+    (effects (font (size 1.4 1.4) (thickness 0.15)) (justify mirror))
+  )
+  (gr_text "Solar\nOUT" (at 81.85 69.8 270) (layer "B.SilkS")
+    (effects (font (size 1.4 1.4) (thickness 0.15)) (justify mirror))
+  )
+  (gr_text "VIN" (at 86.9 63.7) (layer "B.SilkS")
+    (effects (font (size 1.5 1.5) (thickness 0.15)) (justify mirror))
+  )
+  (gr_text "USB\nOUT" (at 81.8 93.1 270) (layer "B.SilkS")
+    (effects (font (size 1.4 1.4) (thickness 0.15)) (justify mirror))
+  )
+  (gr_text "GND" (at 92.1 63.65) (layer "B.SilkS")
+    (effects (font (size 1.5 1.5) (thickness 0.15)) (justify mirror))
+  )
+  (gr_text "Solar\nIN" (at 82 59.65 270) (layer "B.SilkS")
+    (effects (font (size 1.5 1.4) (thickness 0.15)) (justify mirror))
+  )
+  (gr_text "By Andy \n2022/08/08" (at 88.1 87.3) (layer "F.SilkS")
+    (effects (font (size 1.2 1.2) (thickness 0.15)))
+  )
   (via (at 83.9 78.4) (size 0.8) (drill 0.4) (layers "F.Cu" "B.Cu") (net 1))
   (via (at 83.9 72.5) (size 0.8) (drill 0.4) (layers "F.Cu" "B.Cu") (free) (net 1))
@@
         (xy 91.85 79.05)
         (xy 91.85 76.4)
-        (xy 91.85 76.4)
         (xy 91.85 73.4)
