File: Solar charger/CN3795 MPPT.kicad_sch (KiCad schematic)
At the start: 18 parts, among them U1 CN3795

Commit message: board compelet
Parts:
- added R1, R7: 100K, Resistor_SMD:R_0805_2012Metric, symbol Device:R_US
- added R2: 15K, Resistor_SMD:R_0805_2012Metric, symbol Device:R_US
- added R8: 13K, Resistor_SMD:R_0805_2012Metric, symbol Device:R_US
- gave numbers to parts that had none: 17
Connections:
- net FB: now also R1.1, R2.2
- net GND: now also R2.1, R8.1
- net Power Output: now also R1.2
- net VCC: now also R7.2
- net MPPT: now reaches U1.4 (MPPT)
- net MPPT: now also R7.1, R8.2
Other:
- moved on the sheet: C7, C8

Commit message: update
Parts:
- U1: LCSC (none) -> https://lcsc.com/product-detail/Battery-Management-ICs_Shan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
Changed lines of the file:
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@@
+      (effects (font (size 1.27 1.27)) hide)
+    )
+    (property "LCSC" "" (id 4) (at 78.74 69.85 0)
       (effects (font (size 1.27 1.27)) hide)
     )
@@
       (effects (font (size 1.27 1.27)) hide)
     )
+    (property "LCSC" "" (id 4) (at 177.8 73.66 0)
+      (effects (font (size 1.27 1.27)) hide)
+    )
     (pin "1")
     (pin "2")
@@
     )
     (property "Datasheet" "https://datasheet.lcsc.com/lcsc/1912111437_ALLPOWER-ShenZhen-Quan-Li-Semiconductor-AP4435_C353082.pdf" (id 3) (at 170.18 60.96 0)
+      (effects (font (size 1.27 1.27)) hide)
+    )
+    (property "LCSC" "~" (id 4) (at 153.67 60.96 0)
       (effects (font (size 1.27 1.27)) hide)
     )
@@
     )
     (property "Datasheet" "https://datasheet.lcsc.com/lcsc/1810010417_ShangHai-Consonance-Elec-CN3795_C150555.pdf" (id 3) (at 138.43 104.14 0)
+      (effects (font (size 1.27 1.27)) hide)
+    )
+    (property "LCSC" "https://lcsc.com/product-detail/Battery-Management-ICs_ShangHai-Consonance-Elec-CN3795_C150555.html" (id 4) (at 138.43 92.71 0)
       (effects (font (size 1.27 1.27)) hide)
     )
@@
       (effects (font (size 1.27 1.27)) hide)
     )
+    (property "LCSC" "~" (id 4) (at 120.65 67.31 0)
+      (effects (font (size 1.27 1.27)) hide)
+    )
     (pin "1")
     (pin "2")
@@
       (effects (font (size 1.27 1.27)) hide)
     )
+    (property "LCSC" "" (id 4) (at 88.9 69.85 0)
+      (effects (font (size 1.27 1.27)) hide)
+    )

Commit message: 增加電路圖PDF，新增修改一些元件
Other:
- title: (none) -> Solar Power IN CN3795 OUT
Changed lines of the file:
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@@
 (kicad_sch (version 20211123) (generator eeschema)
   (paper "A4")
+  (title_block
+    (title "Solar Power IN CN3795 OUT")
+  )
   (junction (at 186.69 48.26) (diameter 0) (color 0 0 0 0)
   )
