File: Solar charger/Solar Charger.kicad_sch (KiCad schematic)
At the start: 5 parts, among them P1 USB_C_Plug_USB2.0

Commit message: board compelet
Parts:
- J1: renamed from J?; footprint TerminalBlock_Phoenix:TerminalBlock_Phoenix_MKDS-1,5-3-5.08_1x03_P5.08mm_Horizontal -> TerminalBlock:TerminalBlock_bornier-3_P5.08mm
- J2, J3: renamed from J?; footprint TerminalBlock_Phoenix:TerminalBlock_Phoenix_MKDS-1,5-2_1x02_P5.00mm_Horizontal -> TerminalBlock:TerminalBlock_bornier-2_P5.08mm
