File: Circuit/V2/Solar charger/MCU.kicad_sch (KiCad schematic)
At the start: 16 parts, among them J1 Conn_02x05_Odd_Even, SW1 SW_Push, U10 N76E003AT20, U7 NCT3933U, U8 AMS1117-3.3, U9 INA180A3IDBVR

Commit message: update
Parts:
- removed C19: 0.1u, Capacitor_SMD:C_0805_2012Metric, symbol 1CommonUse:C0805
- removed R27: 0.1, Resistor_SMD:R_0805_2012Metric, symbol 1CommonUse:R0805
- removed U9: INA180A3IDBVR, Package_TO_SOT_SMD:SOT-23-5, symbol SolarCharger:INA180A3IDBVR
Connections:
- net +9V: now reaches C17.1, U8.3 (VI)
