File: Circuit/V2/Solar charger/SuperCapacitor.kicad_sch (KiCad schematic)
At the start: 13 parts

Commit message: update
Parts:
- removed C?: 160n, Capacitor_SMD:C_0805_2012Metric, symbol 1CommonUse:C0805
- removed R?: 0.015, Resistor_SMD:R_0805_2012Metric, symbol 1CommonUse:R0805
- removed R? (x2): 5, Resistor_SMD:R_0805_2012Metric, symbol 1CommonUse:R0805
- removed U?: INA180A3IDBVR, Package_TO_SOT_SMD:SOT-23-5, symbol SolarCharger:INA180A3IDBVR
- added C10, C11: LIC1313Q3R8706-10F, Capacitor_THT:CP_Radial_D13.0mm_P5.00mm, symbol Device:C_Polarized
- added C12, C14, C15, C16: 0.1u, Capacitor_SMD:C_0805_2012Metric, symbol 1CommonUse:C0805
- added C13: 1u, Capacitor_SMD:C_0805_2012Metric, symbol 1CommonUse:C0805
- added Q1, Q3: Q_PMOS_GSD, Package_TO_SOT_SMD:SOT-23, symbol Device:Q_PMOS_GSD
- added Q2, Q4: Q_NMOS_GDS, Package_TO_SOT_SMD:SOT-23, symbol Device:Q_NMOS_GDS
- added R12, R13, R14, R19, R20, R8: 100K, Resistor_SMD:R_0805_2012Metric, symbol 1CommonUse:R0805
- added R15, R21: 100k, Resistor_SMD:R_0805_2012Metric, symbol 1CommonUse:R0805
- added R16, R18, R22, R24: 150k, Resistor_SMD:R_0805_2012Metric, symbol 1CommonUse:R0805
- added R17, R23: 250K, Resistor_SMD:R_0805_2012Metric, symbol 1CommonUse:R0805
- added R9: 20k, Resistor_SMD:R_0805_2012Metric, symbol 1CommonUse:R0805
- added U4: 74AHC1G00, symbol 74xGxx:74AHC1G00
- added U5: LM339, symbol Comparator:LM339
- added U6: ME6206A21M3G, Package_TO_SOT_SMD:SOT-23, symbol SolarCharger:ME6206A21M3G
- R10: renamed from R?; value 45k -> 5.25K
- R11: renamed from R?; value 10k -> 1K
- gave numbers to parts that had none: 6
Connections:
- net GND: now also C11.2, C12.2, C13.2, C14.2, C15.2, C16.2, Q2.3 (S), Q4.3 (S), R12.1, R14.1, R22.1, R24.1, U4.3 (GND), U5.12 (V-), U6.1 (VSS)
- net +12V: now reaches C6.1, C7.1, U3.3 (VIN)
- net +12V: now also Q1.2 (S), R19.2, R8.2
- net FB: now reaches R10.1, R11.2
- net FB: now also R9.1; no longer U3.4 (FB)
- net EN0 renamed OverVoltage
- net OverVoltage: now also R19.1, U5.1, U5.2
- net PowerOutput renamed V1
- net V1: now also C10.1, Q3.2 (S), R13.2, R15.2, R17.2, R21.2
- new net: Q4.1 (G), R14.2, U4.4
- new net: Q3.1 (G), Q4.2 (D), R13.1
- new net: R15.1, R16.2, U5.11 (+)
- new net: R17.1, R18.2, U5.4 (-)
- new net: R23.1, R24.2, U5.6 (-)
- new net: R21.1, R22.2, U5.9 (+)
- new net: Q1.1 (G), Q2.2 (D), R8.1
- new net: R9.2, U3.4 (FB)
- new net +9V: C12.1, C13.1, C14.1, Q1.3 (D), Q3.3 (D), R20.2, U5.3 (V+), U6.3 (VI)
- new net 2.5W?: Q2.1 (G), R12.2, U4.1
- new net LowerVoltage: R20.1, U4.2, U5.13, U5.14
- new net V2: C10.2, C11.1, R16.1, R18.1, R23.2
- new net VCC: C15.1, C16.1, U4.5 (VCC), U5.10 (-), U5.5 (+), U5.7 (+), U5.8 (-), U6.2 (VO)
Other:
- moved on the sheet: C6, C7, C8, C9, L2, R10, R11, U3
