File: Circuit/V2/Solar charger/SuperCapacitor.kicad_sch (KiCad schematic)
At the start: 37 parts, among them Q1 Q_PMOS_GSD, Q2 Q_NMOS_GDS, Q3 Q_PMOS_GSD, Q4 Q_NMOS_GDS, U3 BL8032CB6TR, U4 74AHC1G00, U5 LM339, U6 ME6206A21M3G

Commit message: update
Parts:
- added C?: LIC1313Q3R8706-10F, Capacitor_THT:CP_Radial_D13.0mm_P5.00mm, symbol Device:C_Polarized
Connections:
- net V1: no longer R21.2
- net V2: now also R21.2
Changed lines of the file:
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@@
     (effects (font (size 1.27 1.27)) (justify left bottom))
   )
-  (label "V1" (at 276.86 129.54 0)
+  (label "V2" (at 276.86 129.54 0)
     (effects (font (size 1.27 1.27)) (justify left bottom))
   )
@@
     (pin "1")
   )
+  (symbol (lib_id "Device:C_Polarized") (at 71.12 165.1 0) (unit 1)
+    (in_bom yes) (on_board yes)
+    (property "Reference" "C?" (id 0) (at 75.184 162.9409 0)
+      (effects (font (size 1.27 1.27)) (justify left))
+    )
+    (property "Value" "LIC1313Q3R8706-10F" (id 1) (at 61.595 167.005 0)
+      (effects (font (size 1.27 1.27)) (justify left))
+    )
+    (property "Footprint" "Capacitor_THT:CP_Radial_D13.0mm_P5.00mm" (id 2) (at 72.0852 168.91 0)
+      (effects (font (size 1.27 1.27)) hide)
+    )
+    (property "Datasheet" "http://www.cda-cap.com/userfiles/20217301571475.pdf" (id 3) (at 71.12 165.1 0)
+      (effects (font (size 1.27 1.27)) hide)
+    )
+    (property "淘寶" "https://item.taobao.com/item.htm?spm=a312a.7700824.w4002-https://item.taobao.com/item.htm?spm=a312a.7700824.w4002-23251773187.26.64b61871zzsKnK&id=607728818790" (id 4) (at 71.12 165.1 0)
+      (effects (font (size 1.27 1.27)) hide)
+    )
+    (pin "1")
+    (pin "2")
+  )
   (symbol (lib_id "Comparator:LM339") (at 241.3 142.24 0) (unit 3)
