File: Circuit/V2/Solar charger/Type-c.kicad_sch (KiCad schematic)
At the start: 1 part

Commit message: update
Parts:
- added U?: PS9115FS6, Package_TO_SOT_SMD:SOT-23-6, symbol SolarCharger:PS9115FS6
- P?: LCSC (none) -> https://lcsc.com/product-detail/USB-Connectors_Korean-Hropa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
Connections:
- net at P?.A6 (D+): now also U?.1 (DP)
- net at P?.A7 (D-): now also U?.6 (DM)
Other:
- moved on the sheet: P?
Changed lines of the file:
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@@
 (kicad_sch (version 20211123) (generator eeschema)
   (paper "A4")
-  (symbol (lib_id "Connector:USB_C_Plug_USB2.0") (at 84.455 67.945 0) (unit 1)
+  (wire (pts (xy 174.625 92.075) (xy 174.625 102.87))
+    (stroke (width 0) (type default) (color 0 0 0 0))
+  )
+  (wire (pts (xy 174.625 102.87) (xy 172.085 102.87))
+    (stroke (width 0) (type default) (color 0 0 0 0))
+  )
+  (wire (pts (xy 145.415 102.235) (xy 145.415 92.075))
+    (stroke (width 0) (type default) (color 0 0 0 0))
+  )
+  (wire (pts (xy 140.97 107.315) (xy 147.955 107.315))
+    (stroke (width 0) (type default) (color 0 0 0 0))
+  )
+  (wire (pts (xy 147.955 102.87) (xy 154.305 102.87))
+    (stroke (width 0) (type default) (color 0 0 0 0))
+  )
+  (wire (pts (xy 145.415 92.075) (xy 174.625 92.075))
+    (stroke (width 0) (type default) (color 0 0 0 0))
+  )
+  (wire (pts (xy 140.97 102.235) (xy 145.415 102.235))
+    (stroke (width 0) (type default) (color 0 0 0 0))
+  )
+  (wire (pts (xy 147.955 107.315) (xy 147.955 102.87))
+    (stroke (width 0) (type default) (color 0 0 0 0))
+  )
+  (symbol (lib_id "SolarCharger:PS9115FS6") (at 163.195 105.41 0) (unit 1)
     (in_bom yes) (on_board yes) (fields_autoplaced)
-    (property "Reference" "P?" (id 0) (at 84.455 44.45 0))
-    (property "Value" "USB_C_Plug_USB2.0" (id 1) (at 84.455 46.99 0))
-    (property "Footprint" "SolarCharger:USB-C-SMD_TYPE-C-31-E-03" (id 2) (at 88.265 67.945 0)
+    (property "Reference" "U?" (id 0) (at 163.195 95.25 0))
+    (property "Value" "PS9115FS6" (id 1) (at 163.195 97.79 0))
+    (property "Footprint" "Package_TO_SOT_SMD:SOT-23-6" (id 2) (at 163.195 102.743 0)
       (effects (font (size 1.27 1.27)) hide)
     )
-    (property "Datasheet" "https://www.usb.org/sites/default/files/documents/usb_type-c.zip" (id 3) (at 88.265 67.945 0)
+    (property "Datasheet" "http://www.szlcsc.com/product/details_678370.html" (id 3) (at 163.195 107.823 0)
       (effects (font (size 1.27 1.27)) hide)
     )
+    (property "SuppliersPartNumber" "C648908" (id 4) (at 163.195 112.903 0)
+      (effects (font (size 1.27 1.27)) hide)
+    )
+    (property "uuid" "std:6d7a594c6c8842de90c89203bf2a6eec" (id 5) (at 163.195 112.903 0)
+      (effects (font (size 1.27 1.27)) hide)
+    )
+    (pin "1")
+    (pin "2")
+    (pin "3")
+    (pin "4")
+    (pin "5")
+    (pin "6")
+  )
+  (symbol (lib_id "Connector:USB_C_Plug_USB2.0") (at 125.73 104.775 0) (unit 1)
+    (in_bom yes) (on_board yes) (fields_autoplaced)
+    (property "Reference" "P?" (id 0) (at 125.73 81.28 0))
+    (property "Value" "USB_C_Plug_USB2.0" (id 1) (at 125.73 83.82 0))
+    (property "Footprint" "SolarCharger:USB-C-SMD_TYPE-C-31-E-03" (id 2) (at 129.54 104.775 0)
+      (effects (font (size 1.27 1.27)) hide)
+    )
+    (property "Datasheet" "https://www.usb.org/sites/default/files/documents/usb_type-c.zip" (id 3) (at 129.54 104.775 0)
+      (effects (font (size 1.27 1.27)) hide)
+    )
+    (property "LCSC" "https://lcsc.com/product-detail/USB-Connectors_Korean-Hroparts-Elec-TYPE-C-31-E-03_C840342.html" (id 4) (at 125.73 104.775 0)
+      (effects (font (size 1.27 1.27)) hide)
+    )

Commit message: update
Parts:
- added C5: 0.47u, Capacitor_SMD:C_0805_2012Metric, symbol 1CommonUse:C0805
- added R4, R5: 56K, Resistor_SMD:R_0805_2012Metric, symbol 1CommonUse:R0805
- added R6: 2.2k, Resistor_SMD:R_0805_2012Metric, symbol 1CommonUse:R0805
- added R7: 10K, Resistor_SMD:R_0805_2012Metric, symbol 1CommonUse:R0805
- gave numbers to parts that had none: 2
Connections:
- net GND: now reaches U2.2 (GND)
- net GND: now also P1.A1 (GND), P1.A12 (GND), P1.B1 (GND), P1.B12 (GND), P1.S1 (SHIELD), C5.1
- net FB: now reaches U2.3 (FB)
- net at U2.4 (QE): now also R7.2
- net at U2.5 (BP): now also C5.2, R6.2
- net PowerInput: now reaches P1.A4 (VBUS), P1.A9 (VBUS), P1.B4 (VBUS), P1.B9 (VBUS)
- net PowerInput: now also R4.1, R5.1, R6.1, R7.1
- net CC1: now reaches P1.A5 (CC)
- net CC1: now also R4.2
- net CC2: now reaches P1.B5 (VCONN)
- net CC2: now also R5.2
Other:
- moved on the sheet: P1, U2
